File: eagle/quasi_bb_nano_controller.sch (EAGLE design)
At the start: 10 parts, among them X1 JST-XH-08-PIN-LONG-PAD, X2 JST-XH-08-PIN-LONG-PAD, X3 JST-XH-02-PIN-LONG-PAD, X4 JST-XH-08-PIN-LONG-PAD, X5 JST-XH-08-PIN-LONG-PAD

Commit message: update boards
Connections:
- net A1_0: now also U$1.D12; no longer U$1.D8
- net A2_0: now also U$1.D13; no longer U$1.D9
- net B1_0: now also U$1.D8; no longer U$1.D7
- net B2_0: now also U$1.D7; no longer U$1.D6
- net PWMA_0: now also U$1.D11; no longer U$1.D13
- net PWMA_1: now also U$1.D6; no longer U$1.D10
- net PWMB_0: now also U$1.D10; no longer U$1.D12
- net PWMB_1: now also U$1.D9; no longer U$1.D11
