File: eagle/quasi_bb_nano_controller.brd (EAGLE design)
At the start: 62.4 x 70.6 mm, 10 parts, among them X1 JST-XH-08-PIN-LONG-PAD, X2 JST-XH-08-PIN-LONG-PAD, X3 JST-XH-02-PIN-LONG-PAD, X4 JST-XH-08-PIN-LONG-PAD, X5 JST-XH-08-PIN-LONG-PAD

Commit message: update board
Routing:
- net VM: track 65.1 -> 49.8 mm, vias 0 -> 2
- net VCC: track 129.9 -> 131.4 mm, vias 0 -> 3
- net B1_1: track 23.3 -> 24.4 mm
- net A2_0: track 16.8 -> 17.5 mm
- net A1_0: track 20.4 -> 21.1 mm
- net B2_1: track 27.7 -> 28.4 mm
- net PWMA_1: vias 0 -> 2
- net PWMB_1: vias 0 -> 2
- net PWMB_0: vias 0 -> 2
- net PWMA_0: vias 0 -> 2

Commit message: update boards
Connections:
- net A1_0: now also U$1.D12; no longer U$1.D8
- net A2_0: now also U$1.D13; no longer U$1.D9
- net B1_0: now also U$1.D8; no longer U$1.D7
- net B2_0: now also U$1.D7; no longer U$1.D6
- net PWMA_0: now also U$1.D11; no longer U$1.D13
- net PWMA_1: now also U$1.D6; no longer U$1.D10
- net PWMB_0: now also U$1.D10; no longer U$1.D12
- net PWMB_1: now also U$1.D9; no longer U$1.D11
Routing:
- net PWMA_1: track 71.3 -> 20.2 mm
- net A2_0: track 17.5 -> 34.5 mm
- net PWMB_1: track 63.1 -> 53.7 mm
- net PWMA_0: track 25.7 -> 20.4 mm, vias 2 -> 0
- net A1_0: track 21.1 -> 16.9 mm
- net PWMB_0: track 27.2 -> 30.8 mm
- net B2_0: track 32.2 -> 34.1 mm
- net A1_1: track 23.1 -> 24.2 mm
- net B1_0: track 28.4 -> 29.2 mm
- net A2_1: track 19.9 -> 20.5 mm
Other:
- board size 62.4 x 70.6 mm -> 56.8 x 70.6 mm

Commit message: Add eagle
Routing:
- net VCC: track 131.4 -> 0.00 mm, vias 3 -> 0
- added copper zone on layer 1, net VCC
Changed lines of the file:
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@@
 <setting verticaltext="up"/>
 </settings>
-<grid distance="10" unitdist="mil" unit="mil" style="lines" multiple="5" display="yes" altdistance="5" altunitdist="mil" altunit="mil"/>
+<grid distance="0.25" unitdist="inch" unit="inch" style="lines" multiple="1" display="yes" altdistance="5" altunitdist="mil" altunit="inch"/>
 <layers>
 <layer number="1" name="Top" color="4" fill="1" visible="yes" active="yes"/>
@@
 <contactref element="U$1" pad="5V"/>
 <contactref element="X4" pad="2"/>
-<wire x1="16.51" y1="22.86" x2="16.51" y2="35.56" width="0.4064" layer="1"/>
-<wire x1="16.51" y1="22.86" x2="16.51" y2="19.05" width="0.4064" layer="1"/>
-<wire x1="16.51" y1="35.56" x2="16.51" y2="19.05" width="0.6096" layer="1"/>
-<wire x1="20.574" y1="14.986" x2="16.51" y2="19.05" width="0.6096" layer="1"/>
-<wire x1="16.51" y1="22.86" x2="37.338" y2="22.86" width="0.6096" layer="1"/>
-<wire x1="37.338" y1="22.86" x2="37.338" y2="50.546" width="0.6096" layer="1"/>
-<wire x1="41.656" y1="54.864" x2="37.338" y2="50.546" width="0.6096" layer="1"/>
-<wire x1="19.05" y1="35.56" x2="16.51" y2="35.56" width="0.6096" layer="16"/>
-<via x="16.51" y="35.56" extent="1-16" drill="0.8"/>
-<wire x1="45.72" y1="52.07" x2="45.72" y2="54.864" width="0.6096" layer="16"/>
-<via x="45.72" y="54.864" extent="1-16" drill="0.8"/>
-<wire x1="45.72" y1="54.864" x2="41.656" y2="54.864" width="0.6096" layer="1"/>
-<wire x1="45.72" y1="19.05" x2="45.72" y2="16.002" width="0.6096" layer="16"/>
-<via x="45.72" y="16.002" extent="1-16" drill="0.8"/>
-<wire x1="45.72" y1="16.002" x2="44.704" y2="14.986" width="0.6096" layer="1"/>
-<wire x1="44.704" y1="14.986" x2="20.574" y2="14.986" width="0.6096" layer="1"/>
+<polygon width="0.1524" layer="1" isolate="0.8636">
+<vertex x="6.35" y="82.55"/>
+<vertex x="76.2" y="82.55"/>
+<vertex x="76.2" y="0"/>
+<vertex x="6.35" y="0"/>
+</polygon>
+<wire x1="19.05" y1="35.56" x2="45.72" y2="52.07" width="0" layer="19" extent="1-1"/>
+<wire x1="45.72" y1="19.05" x2="19.05" y2="35.56" width="0" layer="19" extent="1-1"/>
 </signal>
 <signal name="GND">
