File: eagle/quasi_bb_nano_controller_3drivers.brd (EAGLE design)
At the start: 62.4 x 70.6 mm, 10 parts, among them X1 JST-XH-08-PIN-LONG-PAD, X2 JST-XH-08-PIN-LONG-PAD, X3 JST-XH-02-PIN-LONG-PAD, X4 JST-XH-08-PIN-LONG-PAD, X5 JST-XH-08-PIN-LONG-PAD

Commit message: Add eagle
Parts:
- added U$6, U$7: JST-PH_2-PIN_HEADER, con-jst-ph:JST_B2B-PH_HEADER
- added X12, X13: JST-XH-03-PIN-LONG-PAD, Rembrandt Electronics - JST XH Connectors v1-0:JST-XH-03-PACKAGE-LONG-PAD
- added X6, X7: JST-XH-08-PIN-LONG-PAD, Rembrandt Electronics - JST XH Connectors v1-0:JST-XH-08-PACKAGE-LONG-PAD
- added X8, X9: JST-XH-04-PIN-LONG-PAD, Rembrandt Electronics - JST XH Connectors v1-0:JST-XH-04-PACKAGE-LONG-PAD
- moved U$4 39.8 mm to (73.9, 45.5), turned to 90 degrees
- moved U$3 35.1 mm to (74.2, 71.1), turned to 90 degrees
- moved U$5 26.9 mm to (74.2, 35.1), turned to 90 degrees
- moved U$2 22.3 mm to (74.2, 61.0), turned to 90 degrees
- moved X5 14.3 mm to (58.2, 47.2)
- moved X4 14.3 mm to (58.2, 32.0)
- moved U$1 8.27 mm to (35.3, 42.4)
- moved X1 8.27 mm to (58.2, 57.7)
- moved X2 8.27 mm to (58.2, 72.9)
- moved X3 6.28 mm to (32.8, 20.6)
Connections:
- removed net N$12: X2.4
- removed net N$121: X5.4
- new net 485_A: X12.1, X13.1, X9.2
- new net 485_B: X12.2, X13.2, X9.3
- new net A0: U$1.A0, X8.4
- new net A01_2: U$6.P1, X6.4
- new net A02_2: U$6.P2, X6.5
- new net A1: U$1.A1, X8.1
- new net A1_2: U$1.A6, X7.3
- new net A2_2: U$1.A7, X7.2
- new net B01_2: U$7.P2, X6.7
- new net B02_2: U$7.P1, X6.6
- new net B1_2: U$1.A5, X7.5
- new net B2_2: U$1.A4, X7.6
- new net PWMA_2: U$1.D3, X7.1
- new net PWMB_2: U$1.D5, X7.7
- net A1_0: now also U$1.D12; no longer U$1.D8
- net A2_0: now also U$1.D13; no longer U$1.D9
- net A2_1: now also U$1.D4; no longer U$1.D3
- net B1_0: now also U$1.D8; no longer U$1.D7
- net B1_1: now also U$1.A2; no longer U$1.D4
- net B2_0: now also U$1.D7; no longer U$1.D6
- net B2_1: now also U$1.A3; no longer U$1.D5
- net GND: now also X12.3, X13.3, X6.3, X6.8, X7.8, X8.2, X8.3, X9.1
- net PWMA_0: now also U$1.D11; no longer U$1.D13
- net PWMA_1: now also U$1.D6; no longer U$1.D10
- net PWMB_0: now also U$1.D10; no longer U$1.D12
- net PWMB_1: now also U$1.D9; no longer U$1.D11
- net VCC: now also X6.2, X9.4
- net VM: now also X6.1
Routing:
- net VCC: track 129.9 -> 0.00 mm
- net B2_2: track 0.00 -> 89.9 mm
- net B1_2: track 0.00 -> 81.2 mm
- net A1_2: track 0.00 -> 69.5 mm
- net A2_2: track 0.00 -> 60.5 mm
- net PWMA_1: track 71.3 -> 12.8 mm
- net PWMB_2: track 0.00 -> 49.6 mm, vias 0 -> 1
- net B1_1: track 23.3 -> 64.2 mm
- net B2_1: track 27.7 -> 67.0 mm
- net PWMA_2: track 0.00 -> 32.6 mm, vias 0 -> 1
- net 485_B: track 0.00 -> 27.7 mm
- net 485_A: track 0.00 -> 27.7 mm
- net A01_2: track 0.00 -> 24.3 mm
- net A1: track 0.00 -> 23.5 mm
- net A02_2: track 0.00 -> 20.8 mm
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- added copper zone on layer 1, net VCC
Other:
- board size 62.4 x 70.6 mm -> 81.2 x 80 mm
- board text added: "Billy Bass Controller v1.0 Royal Palms"
- board text added: "QUASI #001"

Commit message: Control board v1.0
Parts:
- removed U$2, U$3, U$4, U$5, U$6, U$7: JST-PH_2-PIN_HEADER, con-jst-ph:JST_B2B-PH_HEADER
- removed X1, X2, X4, X5, X6, X7: JST-XH-08-PIN-LONG-PAD, Rembrandt Electronics - JST XH Connectors v1-0:JST-XH-08-PACKAGE-LONG-PAD
- removed X12: JST-XH-03-PIN-LONG-PAD, Rembrandt Electronics - JST XH Connectors v1-0:JST-XH-03-PACKAGE-LONG-PAD
- removed X8, X9: JST-XH-04-PIN-LONG-PAD, Rembrandt Electronics - JST XH Connectors v1-0:JST-XH-04-PACKAGE-LONG-PAD
- added (GND), RS485(TX): JST-XH-04-PIN-LONG-PAD, Rembrandt Electronics - JST XH Connectors v1-0:JST-XH-04-PACKAGE-LONG-PAD
- added D1, D1(VM), D2, D2(VM), D3, D3(VM): JST-XH-08-PIN-LONG-PAD, Rembrandt Electronics - JST XH Connectors v1-0:JST-XH-08-PACKAGE-LONG-PAD
- added IN(A): JST-XH-03-PIN-LONG-PAD, Rembrandt Electronics - JST XH Connectors v1-0:JST-XH-03-PACKAGE-LONG-PAD
- added M1(+), M2(+), M3(+), M4(+), M5(+), M6(+): JST-PH_2-PIN_HEADER, con-jst-ph:JST_B2B-PH_HEADER
- added VIN, X10: JST-XH-02-PIN-LONG-PAD, Rembrandt Electronics - JST XH Connectors v1-0:JST-XH-02-PACKAGE-LONG-PAD
- renumbered X13 to OUT(A), X3 to VM(GND)
Connections:
- removed net A0: U$1.A0, X8.4
- removed net A1: U$1.A1, X8.1
- new net RAW1: U$1.RAW, VIN.1
- new net RX1: RS485(TX).4, X10.2
- new net RX2: U$1.RX1, X10.1
- new net TX: RS485(TX).1, U$1.TX0
- net 485_A: now also (GND).2, IN(A).1; no longer X12.1, X9.2
- net 485_B: now also (GND).3, IN(A).2; no longer X12.2, X9.3
- net A01_0: now also D1(VM).4, M1(+).P1; no longer U$3.P1, X1.4
- net A01_1: now also D2(VM).4, M3(+).P1; no longer U$4.P1, X4.4
- net A01_2: now also D3(VM).4, M5(+).P1; no longer U$6.P1, X6.4
- net A02_0: now also D1(VM).5, M1(+).P2; no longer U$3.P2, X1.5
- net A02_1: now also D2(VM).5, M3(+).P2; no longer U$4.P2, X4.5
- net A02_2: now also D3(VM).5, M5(+).P2; no longer U$6.P2, X6.5
- net A1_0: now also D1.3; no longer X2.3
- net A1_1: now also D2.3; no longer X5.3
- net A1_2: now also D3.3, U$1.A4; no longer U$1.A6, X7.3
- net A2_0: now also D1.2; no longer X2.2
- net A2_1: now also D2.2; no longer X5.2
- net A2_2: now also D3.2, U$1.A5; no longer U$1.A7, X7.2
- net B01_0: now also D1(VM).7, M2(+).P2; no longer U$2.P2, X1.7
- net B01_1: now also D2(VM).7, M4(+).P2; no longer U$5.P2, X4.7
- net B01_2: now also D3(VM).7, M6(+).P2; no longer U$7.P2, X6.7
- net B02_0: now also D1(VM).6, M2(+).P1; no longer U$2.P1, X1.6
- net B02_1: now also D2(VM).6, M4(+).P1; no longer U$5.P1, X4.6
- net B02_2: now also D3(VM).6, M6(+).P1; no longer U$7.P1, X6.6
- net B1_0: now also D1.5; no longer X2.5
- net B1_1: now also D2.5; no longer X5.5
- net B1_2: now also D3.5, U$1.A1; no longer U$1.A5, X7.5
- net B2_0: now also D1.6; no longer X2.6
- net B2_1: now also D2.6; no longer X5.6
- net B2_2: now also D3.6, U$1.A0; no longer U$1.A4, X7.6
- net GND: now also (GND).1, D1(VM).3, D1(VM).8, D1.8, D2(VM).3, D2(VM).8, D2.8, D3(VM).3, D3(VM).8, D3.8, IN(A).3, RS485(TX).2, RS485(TX).3; no longer U$1.GND1, X1.3, X1.8, X12.3, X2.8, X4.3, X4.8, X5.8, X6.3, X6.8, X7.8, X8.2, X8.3, X9.1
- net PWMA_0: now also D1.1; no longer X2.1
- net PWMA_1: now also D2.1; no longer X5.1
- net PWMA_2: now also D3.1; no longer X7.1
- net PWMB_0: now also D1.7; no longer X2.7
- net PWMB_1: now also D2.7; no longer X5.7
- net PWMB_2: now also D3.7; no longer X7.7
- net VCC: now also (GND).4, D1(VM).2, D1.4, D2(VM).2, D2.4, D3(VM).2, D3.4; no longer X1.2, X4.2, X6.2, X9.4
- net VM: now also D1(VM).1, D2(VM).1, D3(VM).1, VIN.2; no longer X1.1, X4.1, X6.1
Routing:
- net TX: track 0.00 -> 69.7 mm
- net VM: track 69.2 -> 110.4 mm
- net RX2: track 0.00 -> 41.0 mm
- net A1: track 23.5 -> 0.00 mm
- net RX1: track 0.00 -> 19.8 mm
- net A01_1: track 24.1 -> 42.1 mm
- net B2_2: track 89.9 -> 107.7 mm
- net B1_2: track 81.2 -> 98.0 mm
- net A0: track 14.8 -> 0.00 mm
- net A1_2: track 69.5 -> 82.1 mm
- net A2_2: track 60.5 -> 72.1 mm
- net A2_0: track 34.5 -> 42.2 mm
- net 485_B: track 27.7 -> 21.4 mm
- net 485_A: track 27.7 -> 21.5 mm
- net RAW1: track 0.00 -> 6.13 mm
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Other:
- board size 81.2 x 80 mm -> 84.8 x 80 mm
