File: eagle/quasi_bb_nano_controller_3drivers.sch (EAGLE design)
At the start: 10 parts, among them X1 JST-XH-08-PIN-LONG-PAD, X2 JST-XH-08-PIN-LONG-PAD, X3 JST-XH-02-PIN-LONG-PAD, X4 JST-XH-08-PIN-LONG-PAD, X5 JST-XH-08-PIN-LONG-PAD

Commit message: Add eagle
Parts:
- added U$6, U$7: JST-PH_2-PIN_HEADER, con-jst-ph:JST-PH_2-PIN_HEADER
- added X12, X13: JST-XH-03-PIN-LONG-PAD, Rembrandt Electronics - JST XH Connectors v1-0:JST-XH-03-PIN-LONG-PAD
- added X6, X7: JST-XH-08-PIN-LONG-PAD, Rembrandt Electronics - JST XH Connectors v1-0:JST-XH-08-PIN-LONG-PAD
- added X8, X9: JST-XH-04-PIN-LONG-PAD, Rembrandt Electronics - JST XH Connectors v1-0:JST-XH-04-PIN-LONG-PAD
Connections:
- removed net N$12: X2-4.S
- removed net N$121: X5-4.S
- new net 485_A: X12-1.S, X13-1.S, X9-2.S
- new net 485_B: X12-2.S, X13-2.S, X9-3.S
- new net A0: U$1.A0, X8-4.S
- new net A01_2: U$6.1, X6-4.S
- new net A02_2: U$6.2, X6-5.S
- new net A1: U$1.A1, X8-1.S
- new net A1_2: U$1.A6, X7-3.S
- new net A2_2: U$1.A7, X7-2.S
- new net B01_2: U$7.2, X6-7.S
- new net B02_2: U$7.1, X6-6.S
- new net B1_2: U$1.A5, X7-5.S
- new net B2_2: U$1.A4, X7-6.S
- new net PWMA_2: U$1.D3, X7-1.S
- new net PWMB_2: U$1.D5, X7-7.S
- net A1_0: now also U$1.D12; no longer U$1.D8
- net A1_1: now also U$1.D2
- net A2_0: now also U$1.D13; no longer U$1.D9
- net A2_1: now also U$1.D4
- net B1_0: now also U$1.D8; no longer U$1.D7
- net B1_1: now also U$1.A2; no longer U$1.D4
- net B2_0: now also U$1.D7; no longer U$1.D6
- net B2_1: now also U$1.A3; no longer U$1.D5
- net GND: now also X12-3.S, X13-3.S, X6-3.S, X6-8.S, X7-8.S, X8-2.S, X8-3.S, X9-1.S
- net PWMA_0: now also U$1.D11; no longer U$1.D13
- net PWMA_1: now also U$1.D6; no longer U$1.D10
- net PWMB_0: now also U$1.D10; no longer U$1.D12
- net PWMB_1: now also U$1.D9; no longer U$1.D11
- net VCC: now also X6-2.S, X9-4.S
- net VM: now also X6-1.S

Commit message: Control board v1.0
Parts:
- added VIN, X10: JST-XH-02-PIN-LONG-PAD, Rembrandt Electronics - JST XH Connectors v1-0:JST-XH-02-PIN-LONG-PAD
- renumbered U$2 to M2(+), U$3 to M1(+), U$4 to M3(+), U$5 to M4(+), U$6 to M5(+), U$7 to M6(+), X1 to D1(VM), X12 to IN(A), X13 to OUT(A), X2 to D1, X3 to VM(GND), X4 to D2(VM), X5 to D2, X6 to D3(VM), X7 to D3, X8 to RS485(TX), X9 to (GND)
Connections:
- removed net A0: RS485(TX)-4.S, U$1.A0
- removed net A1: RS485(TX)-1.S, U$1.A1
- new net RAW1: U$1.RAW, VIN-1.S
- new net RX1: RS485(TX)-4.S, X10-2.S
- new net RX2: U$1.RX1, X10-1.S
- new net TX: RS485(TX)-1.S, U$1.TX0
- net A1_2: now also U$1.A4; no longer U$1.A6
- net A2_2: now also U$1.A5; no longer U$1.A7
- net B1_2: now also U$1.A1; no longer U$1.A5
- net B2_2: now also U$1.A0; no longer U$1.A4
- net GND: no longer U$1.GND2
- net VCC: now also D1-4.S, D2-4.S, D3-4.S
- net VM: now also VIN-2.S
